Commit message: 在gazebo中显示机械臂

File: arm_model/robots/arm_model.xacro (robot description, xacro)
@@ -1,17 +1,26 @@
 <?xml version = "1.0"?>
 <robot name="car_model" xmlns:xacro="http://www.ros.org/wiki/xacro">
-    <xacro:property name="arm_1_mass" value="1.0" />
-    <xacro:property name="arm_1_a" value="1.0" />
-    <xacro:property name="arm_1_b" value="1.0" />
+    <xacro:property name="arm_1_mass" value="3.0" />
+    <xacro:property name="arm_1_a" value="0.5" />
+    <xacro:property name="arm_1_b" value="0.5" />
     <xacro:property name="arm_1_c" value="3.0" />
+    <xacro:property name="arm_2_mass" value="1.0" />
+    <xacro:property name="arm_2_a" value="0.5" />
+    <xacro:property name="arm_2_b" value="0.5" />
+    <xacro:property name="arm_2_c" value="1" />
+    <xacro:property name="arm_3_mass" value="1.0" />
+    <xacro:property name="arm_3_a" value="0.5" />
+    <xacro:property name="arm_3_b" value="0.5" />
+    <xacro:property name="arm_3_c" value="1" />
+   <xacro:property name="camera_width" value="0.25" />
     <!-- world_link -->
     <link name="world_link">
     </link>
-    <!-- arm -->
+    <!-- arm1 -->
     <link name="arm_1">
         <collision>
             <origin
-              xyz="0 0 0"
-              rpy="0 0 0" />
+                xyz="0 0 ${arm_1_c / 2}"
+                rpy="0 0 0" />
             <geometry>
                 <box size="${arm_1_a} ${arm_1_b} ${arm_1_c}" />
@@ -20,5 +29,5 @@
         <visual>
             <origin
-                xyz="0 0 0"
+                xyz="0 0 ${arm_1_c / 2}"
                 rpy="0 0 0" />
             <geometry>
@@ -26,24 +35,250 @@
             </geometry>
             <material name="DeepPink" >
-               <color rgba="1 0.0784 0.5764 1" />
-            </material>
-        </visual>
-        <inertial>
-            <origin
-              xyz="0 0 0"
-              rpy="0 0 0" />
-            <mass value="${arm_1_mass}" />
-            <inertia
-            ixx="${arm_1_mass / 12.0 * (arm_1_b*arm_1_b + arm_1_c*arm_1_c)}"
-            ixy="0.0"
-            ixz="0.0"
-            iyy="${arm_1_mass / 12.0 * (arm_1_a*arm_1_a + arm_1_c*arm_1_c)}"
-            iyz="0.0"
-            izz="${arm_1_mass / 12.0 * (arm_1_a*arm_1_a + arm_1_b*arm_1_b)}" />
-        </inertial>
-    </link>
-    <joint name="joint_world" type="fixed">
+                <color rgba="1 0.0784 0.5764 0.5" />
+            </material>
+        </visual>
+        <inertial>
+            <origin
+                xyz="0 0 ${arm_1_c / 2}"
+                rpy="0 0 0" />
+            <mass value="${arm_1_mass / 2}" />
+            <inertia
+                ixx="${arm_1_mass / 12.0 * (arm_1_b*arm_1_b + arm_1_c*arm_1_c)}"
+                ixy="0.0"
+                ixz="0.0"
+                iyy="${arm_1_mass / 12.0 * (arm_1_a*arm_1_a + arm_1_c*arm_1_c)}"
+                iyz="0.0"
+                izz="${arm_1_mass / 12.0 * (arm_1_a*arm_1_a + arm_1_b*arm_1_b)}" />
+        </inertial>
+    </link>
+    <joint name="joint_0_1" type="fixed">
+        <axis xyz="1 0 0" rpy="0 0 0" />
         <parent link="world_link" />
         <child link="arm_1" />
-    </joint>
+        <origin xyz="0 0 0" rpy="0 0 0" />
+        <limit effort="100" velocity="100" />
+        <joint_properties damping="0" friction="0" />
+    </joint>
+    <!-- arm2 -->
+    <link name="arm_2">
+        <collision>
+            <origin
+                xyz="0 0 ${arm_2_c / 2}"
+                rpy="0 0 0" />
+            <geometry>
+                <box size="${arm_2_a} ${arm_2_b} ${arm_2_c}" />
+            </geometry>
+        </collision>
+        <visual>
+            <origin
+                xyz="0 0 ${arm_2_c / 2}"
+                rpy="0 0 0" />
+            <geometry>
+                <box size="${arm_2_a} ${arm_2_b} ${arm_2_c}" />
+            </geometry>
+            <material name="Gold" >
+                <color rgba="1 0.8431 0 0.5" />
+            </material>
+        </visual>
+        <inertial>
+            <origin
+                xyz="0 0 ${arm_2_c}"
+                rpy="0 0 0" />
+            <mass value="${arm_2_mass / 2}" />
+            <inertia
+                ixx="${arm_2_mass / 12.0 * (arm_2_b*arm_2_b + arm_2_c*arm_2_c)}"
+                ixy="0.0"
+                ixz="0.0"
+                iyy="${arm_2_mass / 12.0 * (arm_2_a*arm_2_a + arm_2_c*arm_2_c)}"
+                iyz="0.0"
+                izz="${arm_2_mass / 12.0 * (arm_2_a*arm_2_a + arm_2_b*arm_2_b)}" />
+        </inertial>
+    </link>
+    <joint name="joint_1_2" type="continuous">
+        <axis xyz="1 0 0" rpy="0 0 0" />
+        <parent link="arm_1" />
+        <child link="arm_2" />
+        <origin xyz="0 0 ${arm_1_c}" rpy="0 0 0" />
+        <limit effort="100" velocity="100" />
+        <joint_properties damping="0" friction="0" />
+    </joint>
+    <!-- arm3 -->
+    <link name="arm_3">
+        <collision>
+            <origin
+                xyz="0 0 ${arm_3_c / 2}"
+                rpy="0 0 0" />
+            <geometry>
+                <box size="${arm_3_a} ${arm_3_b} ${arm_3_c}" />
+            </geometry>
+        </collision>
+        <visual>
+            <origin
+                xyz="0 0 ${arm_3_c / 2}"
+                rpy="0 0 0" />
+            <geometry>
+                <box size="${arm_3_a} ${arm_3_b} ${arm_3_c}" />
+            </geometry>
+            <material name="Turquoise" >
+                <color rgba="0.2509 0.8784 0.8156 0.5" />
+            </material>
+        </visual>
+        <inertial>
+            <origin
+                xyz="0 0 ${arm_3_c}"
+                rpy="0 0 0" />
+            <mass value="${arm_3_mass / 2}" />
+            <inertia
+                ixx="${arm_3_mass / 12.0 * (arm_3_b*arm_3_b + arm_3_c*arm_3_c)}"
+                ixy="0.0"
+                ixz="0.0"
+                iyy="${arm_3_mass / 12.0 * (arm_3_a*arm_3_a + arm_3_c*arm_3_c)}"
+                iyz="0.0"
+                izz="${arm_3_mass / 12.0 * (arm_3_a*arm_3_a + arm_3_b*arm_3_b)}" />
+        </inertial>
+    </link>
+    <joint name="joint_2_3" type="continuous">
+        <axis xyz="1 0 0" rpy="0 0 0" />
+        <parent link="arm_2" />
+        <child link="arm_3" />
+        <origin xyz="0 0 ${arm_2_c}" rpy="0 0 0" />
+        <limit effort="100" velocity="100" />
+        <joint_properties damping="0" friction="0" />
+    </joint>
+    <!-- camera -->
+    <link name="camera_link">
+        <collision>
+            <origin
+                xyz="0 0 ${arm_3_c}"
+                rpy="0 0 0" />
+            <geometry>
+	            <box size="${camera_width} ${camera_width} ${camera_width}"/>
+            </geometry>
+        </collision>
+        <visual>
+            <origin
+                xyz="0 0 ${arm_3_c}"
+                rpy="0 0 0" />
+            <geometry>
+	            <box size="${camera_width} ${camera_width} ${camera_width}"/>
+            </geometry>
+            <material name="red">
+                <color rgba="0.8 0 0 1"/>
+            </material>
+        </visual>
+        <inertial>
+            <origin
+                xyz="0 0 ${arm_3_c}"
+                rpy="0 0 0"/>
+            <mass value="1.0" />
+            <inertia
+                ixx="1.0"
+                ixy="0"
+                ixz="0"
+                iyy="1.0"
+                iyz="0"
+                izz="1.0" />
+        </inertial>
+    </link>
+    <joint name="joint_camera_link" type="fixed">
+        <axis xyz="1 0 0" rpy="0 0 0" />
+        <origin xyz="0 0 0" rpy="0 0 0"/>
+        <parent link="arm_3"/>
+        <child link="camera_link"/>
+    </joint>
+    <!-- gazebo reference -->
+    <gazebo reference="world_link">
+        <material>Gazebo/Orange</material>
+    </gazebo>
+    <gazebo reference="arm_1">
+        <mu1>0.2</mu1>
+        <mu2>0.2</mu2>
+        <material>Gazebo/Green</material>
+    </gazebo>
+    <gazebo reference="arm_2">
+        <mu1>0.2</mu1>
+        <mu2>0.2</mu2>
+        <material>Gazebo/Yellow</material>
+    </gazebo>
+    <gazebo reference="arm_3">
+        <mu1>0.2</mu1>
+        <mu2>0.2</mu2>
+        <material>Gazebo/Orange</material>
+    </gazebo>
+    <gazebo reference="camera_link">
+        <mu1>0.2</mu1>
+        <mu2>0.2</mu2>
+        <material>Gazebo/Red</material>
+    </gazebo>
+    <!-- transmission -->
+    <transmission name="tran_1_2">
+        <type>transmission_interface/SimpleTransmission</type>
+        <joint name="joint_1_2">
+            <hardwareInterface>hardware_interface/EffortJointInterface</hardwareInterface>
+        </joint>
+        <actuator name="motor_1_2">
+            <hardwareInterface>hardware_interface/EffortJointInterface</hardwareInterface>
+            <mechanicalReduction>1</mechanicalReduction>
+            <motorTorqueConstant>1</motorTorqueConstant>
+        </actuator>
+    </transmission>
+    <transmission name="tran_2_3">
+        <type>transmission_interface/SimpleTransmission</type>
+        <joint name="joint_2_3">
+            <hardwareInterface>hardware_interface/EffortJointInterface</hardwareInterface>
+        </joint>
+        <actuator name="motor_2_3">
+            <hardwareInterface>hardware_interface/EffortJointInterface</hardwareInterface>
+            <mechanicalReduction>1</mechanicalReduction>
+            <motorTorqueConstant>1</motorTorqueConstant>
+        </actuator>
+    </transmission>
+    <gazebo reference="camera_link">
+        <sensor type="camera" name="camera1">
+            <update_rate>30.0</update_rate>
+            <camera name="head">
+                <horizontal_fov>1.3962634</horizontal_fov>
+                <image>
+                    <width>800</width>
+                    <height>800</height>
+                    <format>R8G8B8</format>
+                </image>
+                <clip>
+                    <near>0.02</near>
+                    <far>300</far>
+                </clip>
+                <noise>
+                    <type>gaussian</type>
+                    <mean>0.0</mean>
+                    <stddev>0.007</stddev>
+                </noise>
+            </camera>
+            <plugin name="camera_controller"
+                filename="libgazebo_ros_camera.so">
+                <alwaysOn>true</alwaysOn>
+                <updateRate>0.0</updateRate>
+                <cameraName>rrbot/camera1</cameraName>
+                <imageTopicName>image_raw</imageTopicName>
+                <cameraInfoTopicName>camera_info</cameraInfoTopicName>
+                <frameName>camera_link_optical</frameName>
+                <hackBaseline>0.0</hackBaseline>
+                <distortionK1>0.0</distortionK1>
+                <distortionK2>0.0</distortionK2>
+                <distortionK3>0.0</distortionK3>
+                <distortionT1>0.0</distortionT1>
+                <distortionT2>0.0</distortionT2>
+                <CxPrime>0</CxPrime>
+                <Cx>0.0</Cx>
+                <Cy>0.0</Cy>
+                <focalLength>0.0</focalLength>
+            </plugin>
+        </sensor>
+    </gazebo>
+    <gazebo>
+        <plugin name="gazebo_ros_control"
+            filename="libgazebo_ros_control.so">
+            <robotNamespace>/arm_model</robotNamespace>
+            <robotSimType>gazebo_ros_control/DefaultRobotHWSim</robotSimType>
+        </plugin>
+    </gazebo>
 </robot>

Commit message: 建立五个关节部件

File: arm_model/robots/arm_model.xacro (robot description, xacro)
@@ -13,7 +13,35 @@
     <xacro:property name="arm_3_b" value="0.5" />
     <xacro:property name="arm_3_c" value="1" />
-   <xacro:property name="camera_width" value="0.25" />
+    <xacro:property name="arm_4_mass" value="1.0" />
+    <xacro:property name="arm_4_a" value="0.5" />
+    <xacro:property name="arm_4_b" value="0.5" />
+    <xacro:property name="arm_4_c" value="1" />
+    <xacro:property name="arm_5_mass" value="1.0" />
+    <xacro:property name="arm_5_a" value="0.5" />
+    <xacro:property name="arm_5_b" value="0.5" />
+    <xacro:property name="arm_5_c" value="1" />
+    <xacro:property name="camera_width" value="0.25" />
     <!-- world_link -->
-    <link name="world_link">
+    <link name="base_link">
+        <inertial>
+            <origin xyz="0 0 0" rpy="0 0 0" />
+            <mass value="100" />
+            <inertia ixx="10" ixy="0.0" ixz="0.0" iyy="10" iyz="0.0" izz="10" />
+        </inertial>
+        <visual>
+            <origin xyz="0 0 0" rpy="0 0 0" />
+            <geometry>
+                <box size="10 10 0.1" />
+            </geometry>
+            <material name="Grey">
+                <color rgba="0.79216 0.81961 0.93333 1" />
+            </material>
+        </visual>
+        <collision>
+            <origin xyz="0 0 0" rpy="0 0 0" />
+            <geometry>
+                <box size="10 10 0.1" />
+            </geometry>
+        </collision>
     </link>
     <!-- arm1 -->
@@ -52,7 +80,7 @@
         </inertial>
     </link>
-    <joint name="joint_0_1" type="fixed">
-        <axis xyz="1 0 0" rpy="0 0 0" />
-        <parent link="world_link" />
+    <joint name="joint_0_1" type="continuous">
+        <axis xyz="0 0 1" rpy="0 0 0" />
+        <parent link="base_link" />
         <child link="arm_1" />
         <origin xyz="0 0 0" rpy="0 0 0" />
@@ -146,9 +174,95 @@
         <joint_properties damping="0" friction="0" />
     </joint>
+    <!-- arm4 -->
+    <link name="arm_4">
+        <collision>
+            <origin
+                xyz="0 0 ${arm_4_c / 2}"
+                rpy="0 0 0" />
+            <geometry>
+                <box size="${arm_4_a} ${arm_4_b} ${arm_4_c}" />
+            </geometry>
+        </collision>
+        <visual>
+            <origin
+                xyz="0 0 ${arm_4_c / 2}"
+                rpy="0 0 0" />
+            <geometry>
+                <box size="${arm_4_a} ${arm_4_b} ${arm_4_c}" />
+            </geometry>
+            <material name="Auqamarin" >
+                <color rgba="0.4980 1 0.6666 0.5" />
+            </material>
+        </visual>
+        <inertial>
+            <origin
+                xyz="0 0 ${arm_4_c}"
+                rpy="0 0 0" />
+            <mass value="${arm_4_mass / 2}" />
+            <inertia
+                ixx="${arm_4_mass / 12.0 * (arm_4_b*arm_4_b + arm_4_c*arm_4_c)}"
+                ixy="0.0"
+                ixz="0.0"
+                iyy="${arm_4_mass / 12.0 * (arm_4_a*arm_4_a + arm_4_c*arm_4_c)}"
+                iyz="0.0"
+                izz="${arm_4_mass / 12.0 * (arm_4_a*arm_4_a + arm_4_b*arm_4_b)}" />
+        </inertial>
+    </link>
+    <joint name="joint_3_4" type="continuous">
+        <axis xyz="0 0 1" rpy="0 0 0" />
+        <parent link="arm_3" />
+        <child link="arm_4" />
+        <origin xyz="0 0 ${arm_3_c}" rpy="0 0 0" />
+        <limit effort="100" velocity="100" />
+        <joint_properties damping="0" friction="0" />
+    </joint>
+    <!-- arm5 -->
+    <link name="arm_5">
+        <collision>
+            <origin
+                xyz="0 0 ${arm_5_c / 2}"
+                rpy="0 0 0" />
+            <geometry>
+                <box size="${arm_5_a} ${arm_5_b} ${arm_5_c}" />
+            </geometry>
+        </collision>
+        <visual>
+            <origin
+                xyz="0 0 ${arm_5_c / 2}"
+                rpy="0 0 0" />
+            <geometry>
+                <box size="${arm_5_a} ${arm_5_b} ${arm_5_c}" />
+            </geometry>
+            <material name="Tomato" >
+                <color rgba="1 0.3882 0.2784 0.5" />
+            </material>
+        </visual>
+        <inertial>
+            <origin
+                xyz="0 0 ${arm_5_c}"
+                rpy="0 0 0" />
+            <mass value="${arm_5_mass / 2}" />
+            <inertia
+                ixx="${arm_5_mass / 12.0 * (arm_5_b*arm_5_b + arm_5_c*arm_5_c)}"
+                ixy="0.0"
+                ixz="0.0"
+                iyy="${arm_5_mass / 12.0 * (arm_5_a*arm_5_a + arm_5_c*arm_5_c)}"
+                iyz="0.0"
+                izz="${arm_5_mass / 12.0 * (arm_5_a*arm_5_a + arm_5_b*arm_5_b)}" />
+        </inertial>
+    </link>
+    <joint name="joint_4_5" type="continuous">
+        <axis xyz="1 0 0" rpy="0 0 0" />
+        <parent link="arm_4" />
+        <child link="arm_5" />
+        <origin xyz="0 0 ${arm_4_c}" rpy="0 0 0" />
+        <limit effort="100" velocity="100" />
+        <joint_properties damping="0" friction="0" />
+    </joint>
     <!-- camera -->
     <link name="camera_link">
         <collision>
             <origin
-                xyz="0 0 ${arm_3_c}"
+                xyz="0 0 ${arm_5_c}"
                 rpy="0 0 0" />
             <geometry>
@@ -158,5 +272,5 @@
         <visual>
             <origin
-                xyz="0 0 ${arm_3_c}"
+                xyz="0 0 ${arm_5_c}"
                 rpy="0 0 0" />
             <geometry>
@@ -169,5 +283,5 @@
         <inertial>
             <origin
-                xyz="0 0 ${arm_3_c}"
+                xyz="0 0 ${arm_5_c}"
                 rpy="0 0 0"/>
             <mass value="1.0" />
@@ -184,26 +298,33 @@
         <axis xyz="1 0 0" rpy="0 0 0" />
         <origin xyz="0 0 0" rpy="0 0 0"/>
-        <parent link="arm_3"/>
+        <parent link="arm_5"/>
         <child link="camera_link"/>
     </joint>
     <!-- gazebo reference -->
-    <gazebo reference="world_link">
+    <gazebo reference="arm_1">
+        <mu1>0.2</mu1>
+        <mu2>0.2</mu2>
+        <material>Gazebo/Green</material>
+    </gazebo>
+    <gazebo reference="arm_2">
+        <mu1>0.2</mu1>
+        <mu2>0.2</mu2>
+        <material>Gazebo/Yellow</material>
+    </gazebo>
+    <gazebo reference="arm_3">
+        <mu1>0.2</mu1>
+        <mu2>0.2</mu2>
         <material>Gazebo/Orange</material>
     </gazebo>
-    <gazebo reference="arm_1">
+    <gazebo reference="arm_4">
+        <mu1>0.2</mu1>
+        <mu2>0.2</mu2>
+        <material>Gazebo/Yellow</material>
+    </gazebo>
+    <gazebo reference="arm_5">
         <mu1>0.2</mu1>
         <mu2>0.2</mu2>
         <material>Gazebo/Green</material>
     </gazebo>
-    <gazebo reference="arm_2">
-        <mu1>0.2</mu1>
-        <mu2>0.2</mu2>
-        <material>Gazebo/Yellow</material>
-    </gazebo>
-    <gazebo reference="arm_3">
-        <mu1>0.2</mu1>
-        <mu2>0.2</mu2>
-        <material>Gazebo/Orange</material>
-    </gazebo>
     <gazebo reference="camera_link">
         <mu1>0.2</mu1>
@@ -212,4 +333,15 @@
     </gazebo>
     <!-- transmission -->
+    <transmission name="tran_0_1">
+        <type>transmission_interface/SimpleTransmission</type>
+        <joint name="joint_0_1">
+            <hardwareInterface>hardware_interface/EffortJointInterface</hardwareInterface>
+        </joint>
+        <actuator name="motor_0_1">
+            <hardwareInterface>hardware_interface/EffortJointInterface</hardwareInterface>
+            <mechanicalReduction>1</mechanicalReduction>
+            <motorTorqueConstant>1</motorTorqueConstant>
+        </actuator>
+    </transmission>
     <transmission name="tran_1_2">
         <type>transmission_interface/SimpleTransmission</type>
@@ -229,4 +361,26 @@
         </joint>
         <actuator name="motor_2_3">
+            <hardwareInterface>hardware_interface/EffortJointInterface</hardwareInterface>
+            <mechanicalReduction>1</mechanicalReduction>
+            <motorTorqueConstant>1</motorTorqueConstant>
+        </actuator>
+    </transmission>
+    <transmission name="tran_3_4">
+        <type>transmission_interface/SimpleTransmission</type>
+        <joint name="joint_3_4">
+            <hardwareInterface>hardware_interface/EffortJointInterface</hardwareInterface>
+        </joint>
+        <actuator name="motor_3_4">
+            <hardwareInterface>hardware_interface/EffortJointInterface</hardwareInterface>
+            <mechanicalReduction>1</mechanicalReduction>
+            <motorTorqueConstant>1</motorTorqueConstant>
+        </actuator>
+    </transmission>
+    <transmission name="tran_4_5">
+        <type>transmission_interface/SimpleTransmission</type>
+        <joint name="joint_4_5">
+            <hardwareInterface>hardware_interface/EffortJointInterface</hardwareInterface>
+        </joint>
+        <actuator name="motor_4_5">
             <hardwareInterface>hardware_interface/EffortJointInterface</hardwareInterface>
             <mechanicalReduction>1</mechanicalReduction>
@@ -280,4 +434,5 @@
             <robotNamespace>/arm_model</robotNamespace>
             <robotSimType>gazebo_ros_control/DefaultRobotHWSim</robotSimType>
+            <legacyModeNS>true</legacyModeNS>
         </plugin>
     </gazebo>
